File: barrel-panel-5mm5x2mm1-to-screw-3mm5/barrel-panel-5mm5x2mm1-to-screw-3mm5.kicad_sch (KiCad schematic)
At the start: 1 part, among them J1 Barrel_Jack

Commit message: some updates to barrel connector footprint
Parts:
- J1: footprint Connector_BarrelJack:BarrelJack_SwitchcraftConxall_RAPC10U_Horizontal -> Connector_Barreljack_panel:BarrelJack_panel_5.5mmx2.1mm_2_pins
Changed lines of the file:
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@@
     (property "Reference" "J1" (id 0) (at 118.11 81.28 0))
     (property "Value" "Barrel_Jack" (id 1) (at 118.11 83.82 0))
-    (property "Footprint" "Connector_BarrelJack:BarrelJack_SwitchcraftConxall_RAPC10U_Horizontal" (id 2) (at 119.38 91.186 0)
+    (property "Footprint" "Connector_Barreljack_panel:BarrelJack_panel_5.5mmx2.1mm_2_pins" (id 2) (at 119.38 91.186 0)
       (effects (font (size 1.27 1.27)) hide)
     )
@@
   (symbol_instances
     (path "/68118650-38ea-42b4-9fa0-d2afa9698f5c"
-      (reference "J1") (unit 1) (value "Barrel_Jack") (footprint "Connector_BarrelJack:BarrelJack_SwitchcraftConxall_RAPC10U_Horizontal")
+      (reference "J1") (unit 1) (value "Barrel_Jack") (footprint "Connector_Barreljack_panel:BarrelJack_panel_5.5mmx2.1mm_2_pins")
     )
   )
